Commit message: Add left leg description
TODO: maybe fix link names

File: biped_description/urdf/biped.urdf.xacro (robot description, xacro)
@@ -1,7 +1,10 @@
 <?xml version="1.0"?>
 <robot xmlns:xacro="http://www.ros.org/wiki/xacro" name="biped">
-    <xacro:property name="width" value="0.2" />
-    <xacro:property name="bodylen" value="0.6" />
-    <xacro:property name="leglen" value="0.6" />
+    <material name="red">
+        <color rgba="0.8 0 0 1"/>
+    </material>
+    <material name="green">
+        <color rgba="0 0.8 0 1"/>
+    </material>
     <material name="blue">
         <color rgba="0 0 0.8 1"/>
@@ -10,48 +13,104 @@
         <color rgba="1 1 1 1" />
     </material>
-    <xacro:macro name="leg" params="prefix reflect">
-        <link name="${prefix}_leg">
-            <visual>
-                <geometry>
-                    <box size="${leglen} 0.1 0.2" />
-                </geometry>
-                <origin rpy="0 ${pi/2} 0" xyz="0 0 -${leglen/2}" />
-                <material name="white"/>
-            </visual>
-            <collision>
-                <geometry>
-                    <box size="${leglen} 0.1 0.2" />
-                </geometry>
-                <origin rpy="0 ${pi/2} 0" xyz="0 0 -${leglen/2}" />
-            </collision>
-        </link>
-        <joint name="base_to_${prefix}_leg" type="revolute">
-            <axis xyz="0 1 0"/>
-            <limit effort="5.0" lower="-1.57075" upper="1.57075" velocity="10.0" />
-            <dynamics friction="0.0" damping="0.0" />
-            <parent link="base_link"/>
-            <child link="${prefix}_leg" />
-            <origin xyz="0 ${reflect*(width+0.02)} 0.25" />
-        </joint>
-    </xacro:macro>
+    <material name="black">
+        <color rgba="0 0 0 1" />
+    </material>
+    <xacro:property name="biped_waist_height" value="0.75" />
     <link name="base_link">
+    </link>
+    <link name="l_pelvis_yaw_link">
+    </link>
+    <link name="l_pelvis_roll_link">
+    </link>
+    <link name="l_pelvis_pitch_link">
+    </link>
+    <joint name="l_pelvis_yaw" type="revolute">
+        <axis xyz="0 0 1" />
+        <limit effort="5.0" lower="-${pi/3}" upper="${pi/3}" velocity="5.0" />
+        <origin xyz="0 -0.25 0" rpy="0 0 0" />
+        <parent link="base_link" />
+        <child link="l_pelvis_yaw_link" />
+    </joint>
+    <joint name="l_pelvis_roll" type="revolute">
+        <axis xyz="1 0 0" />
+        <limit effort="5.0" lower="-${pi/3}" upper="${pi/3}" velocity="5.0" />
+        <origin xyz="0 0 0" rpy="0 0 0" />
+        <parent link="l_pelvis_yaw_link" />
+        <child link="l_pelvis_roll_link" />
+    </joint>
+    <joint name="l_pelvis_pitch" type="revolute">
+        <axis xyz="0 1 0" />
+        <limit effort="5.0" lower="-${pi/3}" upper="${pi/3}" velocity="5.0" />
+        <origin xyz="0 0 0" rpy="0 0 0" />
+        <parent link="l_pelvis_roll_link" />
+        <child link="l_pelvis_pitch_link" />
+    </joint>
+    <link name="l_knee_link">
         <visual>
+            <origin xyz="0 0 0.25"/>
             <geometry>
-                <cylinder length="${bodylen}" radius="${width}" />
+                <cylinder radius="0.02" length="0.5" />
             </geometry>
             <material name="blue"/>
         </visual>
-        <collision>
+    </link>
+    <link name="l_knee_pitch_link">
+    </link>
+    <joint name="l_knee_fixed" type="fixed">
+        <origin xyz="0 0 -0.5" rpy="0 0 0" />
+        <parent link="l_pelvis_pitch_link" />
+        <child link="l_knee_link" />
+    </joint>
+    <joint name="l_knee_pitch" type="revolute">
+        <axis xyz="0 1 0" />
+        <limit effort="5.0" lower="0" upper="${pi/2}" velocity="5.0" />
+        <origin xyz="0 0 0" rpy="0 0 0" />
+        <parent link="l_knee_link" />
+        <child link="l_knee_pitch_link" />
+    </joint>
+    <link name="l_ankle_link">
+        <visual>
+            <origin xyz="0 0 0.25"/>
             <geometry>
-                <cylinder length="${bodylen}" radius="${width}" />
+                <cylinder radius="0.02" length="0.5" />
             </geometry>
-        </collision>
-        <inertial>
-            <mass value="10" />
-            <inertia ixx="0.4" ixy="0.0" ixz="0.0" iyy="0.4" iyz="0.0" izz="0.2" />
-            <contact_coefficients mu="0.1" kp="0.0" kd="0.0"/>
-        </inertial>
+            <material name="blue"/>
+        </visual>
     </link>
-    <xacro:leg prefix="right" reflect="-1" />
-    <xacro:leg prefix="left" reflect="1" />
+    <joint name="l_ankle_fixed" type="fixed">
+        <origin xyz="0 0 -0.5" rpy="0 0 0" />
+        <parent link="l_knee_pitch_link" />
+        <child link="l_ankle_link" />
+    </joint>
+    <link name="l_ankle_pitch_link">
+    </link>
+    <joint name="l_ankle_pitch" type="revolute">
+        <axis xyz="0 1 0" />
+        <limit effort="5.0" lower="-${pi/3}" upper="${pi/3}" velocity="5.0" />
+        <origin xyz="0 0 0" rpy="0 0 0" />
+        <parent link="l_ankle_link" />
+        <child link="l_ankle_pitch_link" />
+    </joint>
+    <link name="l_ankle_roll_link">
+    </link>
+    <joint name="l_ankle_roll" type="revolute">
+        <axis xyz="1 0 0" />
+        <limit effort="5.0" lower="-${pi/3}" upper="${pi/3}" velocity="5.0" />
+        <origin xyz="0 0 0" rpy="0 0 0" />
+        <parent link="l_ankle_pitch_link" />
+        <child link="l_ankle_roll_link" />
+    </joint>
+    <link name="l_foot_link">
+        <visual>
+            <origin xyz="0.07 0 0"/>
+            <geometry>
+                <box size="0.3 0.1 0.02" />
+            </geometry>
+        </visual>
+    </link>
+    <joint name="l_foot_fixed" type="fixed">
+        <origin xyz="0 0 0"/>
+        <parent link="l_ankle_roll_link" />
+        <child link="l_foot_link" />
+    </joint>
 </robot>

Commit message: Fix leg TF link names

File: biped_description/urdf/biped.urdf.xacro (robot description, xacro)
@@ -16,101 +16,90 @@
         <color rgba="0 0 0 1" />
     </material>
-    <xacro:property name="biped_waist_height" value="0.75" />
     <link name="base_link">
     </link>
-    <link name="l_pelvis_yaw_link">
-    </link>
-    <link name="l_pelvis_roll_link">
-    </link>
-    <link name="l_pelvis_pitch_link">
-    </link>
-    <joint name="l_pelvis_yaw" type="revolute">
-        <axis xyz="0 0 1" />
-        <limit effort="5.0" lower="-${pi/3}" upper="${pi/3}" velocity="5.0" />
-        <origin xyz="0 -0.25 0" rpy="0 0 0" />
-        <parent link="base_link" />
-        <child link="l_pelvis_yaw_link" />
-    </joint>
-    <joint name="l_pelvis_roll" type="revolute">
-        <axis xyz="1 0 0" />
-        <limit effort="5.0" lower="-${pi/3}" upper="${pi/3}" velocity="5.0" />
-        <origin xyz="0 0 0" rpy="0 0 0" />
-        <parent link="l_pelvis_yaw_link" />
-        <child link="l_pelvis_roll_link" />
-    </joint>
-    <joint name="l_pelvis_pitch" type="revolute">
-        <axis xyz="0 1 0" />
-        <limit effort="5.0" lower="-${pi/3}" upper="${pi/3}" velocity="5.0" />
-        <origin xyz="0 0 0" rpy="0 0 0" />
-        <parent link="l_pelvis_roll_link" />
-        <child link="l_pelvis_pitch_link" />
-    </joint>
-    <link name="l_knee_link">
-        <visual>
-            <origin xyz="0 0 0.25"/>
-            <geometry>
-                <cylinder radius="0.02" length="0.5" />
-            </geometry>
-            <material name="blue"/>
-        </visual>
-    </link>
-    <link name="l_knee_pitch_link">
-    </link>
-    <joint name="l_knee_fixed" type="fixed">
-        <origin xyz="0 0 -0.5" rpy="0 0 0" />
-        <parent link="l_pelvis_pitch_link" />
-        <child link="l_knee_link" />
-    </joint>
-    <joint name="l_knee_pitch" type="revolute">
-        <axis xyz="0 1 0" />
-        <limit effort="5.0" lower="0" upper="${pi/2}" velocity="5.0" />
-        <origin xyz="0 0 0" rpy="0 0 0" />
-        <parent link="l_knee_link" />
-        <child link="l_knee_pitch_link" />
-    </joint>
-    <link name="l_ankle_link">
-        <visual>
-            <origin xyz="0 0 0.25"/>
-            <geometry>
-                <cylinder radius="0.02" length="0.5" />
-            </geometry>
-            <material name="blue"/>
-        </visual>
-    </link>
-    <joint name="l_ankle_fixed" type="fixed">
-        <origin xyz="0 0 -0.5" rpy="0 0 0" />
-        <parent link="l_knee_pitch_link" />
-        <child link="l_ankle_link" />
-    </joint>
-    <link name="l_ankle_pitch_link">
-    </link>
-    <joint name="l_ankle_pitch" type="revolute">
-        <axis xyz="0 1 0" />
-        <limit effort="5.0" lower="-${pi/3}" upper="${pi/3}" velocity="5.0" />
-        <origin xyz="0 0 0" rpy="0 0 0" />
-        <parent link="l_ankle_link" />
-        <child link="l_ankle_pitch_link" />
-    </joint>
-    <link name="l_ankle_roll_link">
-    </link>
-    <joint name="l_ankle_roll" type="revolute">
-        <axis xyz="1 0 0" />
-        <limit effort="5.0" lower="-${pi/3}" upper="${pi/3}" velocity="5.0" />
-        <origin xyz="0 0 0" rpy="0 0 0" />
-        <parent link="l_ankle_pitch_link" />
-        <child link="l_ankle_roll_link" />
-    </joint>
-    <link name="l_foot_link">
-        <visual>
-            <origin xyz="0.07 0 0"/>
-            <geometry>
-                <box size="0.3 0.1 0.02" />
-            </geometry>
-        </visual>
-    </link>
-    <joint name="l_foot_fixed" type="fixed">
-        <origin xyz="0 0 0"/>
-        <parent link="l_ankle_roll_link" />
-        <child link="l_foot_link" />
-    </joint>
+    <xacro:macro name="biped_leg" params="parent_link prefix reflect">
+        <link name="${prefix}_pelvis_yaw_link">
+        </link>
+        <link name="${prefix}_pelvis_roll_link">
+        </link>
+        <link name="${prefix}_pelvis_pitch_link">
+            <visual>
+                <origin xyz="0 0 -0.20"/>
+                <geometry>
+                    <cylinder radius="0.02" length="0.5" />
+                </geometry>
+                <material name="blue"/>
+            </visual>
+        </link>
+        <joint name="${prefix}_pelvis_yaw" type="revolute">
+            <axis xyz="0 0 1" />
+            <limit effort="5.0" lower="-${pi/3}" upper="${pi/3}" velocity="5.0" />
+            <origin xyz="0 ${reflect*0.25} 0" rpy="0 0 0" />
+            <parent link="${parent_link}" />
+            <child link="${prefix}_pelvis_yaw_link" />
+        </joint>
+        <joint name="${prefix}_pelvis_roll" type="revolute">
+            <axis xyz="1 0 0" />
+            <limit effort="5.0" lower="-${pi/3}" upper="${pi/3}" velocity="5.0" />
+            <origin xyz="0 0 0" rpy="0 0 0" />
+            <parent link="${prefix}_pelvis_yaw_link" />
+            <child link="${prefix}_pelvis_roll_link" />
+        </joint>
+        <joint name="${prefix}_pelvis_pitch" type="revolute">
+            <axis xyz="0 1 0" />
+            <limit effort="5.0" lower="-${pi/3}" upper="${pi/3}" velocity="5.0" />
+            <origin xyz="0 0 0" rpy="0 0 0" />
+            <parent link="${prefix}_pelvis_roll_link" />
+            <child link="${prefix}_pelvis_pitch_link" />
+        </joint>
+        <link name="${prefix}_knee_pitch_link">
+            <visual>
+                <origin xyz="0 0 -0.25"/>
+                <geometry>
+                    <cylinder radius="0.02" length="0.5" />
+                </geometry>
+                <material name="red"/>
+            </visual>
+        </link>
+        <joint name="${prefix}_knee_pitch" type="revolute">
+            <axis xyz="0 1 0" />
+            <limit effort="5.0" lower="0" upper="${pi/2}" velocity="5.0" />
+            <origin xyz="0 0 -0.5" rpy="0 0 0" />
+            <parent link="${prefix}_pelvis_pitch_link" />
+            <child link="${prefix}_knee_pitch_link" />
+        </joint>
+        <link name="${prefix}_ankle_pitch_link">
+        </link>
+        <joint name="${prefix}_ankle_pitch" type="revolute">
+            <axis xyz="0 1 0" />
+            <limit effort="5.0" lower="-${pi/3}" upper="${pi/3}" velocity="5.0" />
+            <origin xyz="0 0 -0.5" rpy="0 0 0" />
+            <parent link="${prefix}_knee_pitch_link" />
+            <child link="${prefix}_ankle_pitch_link" />
+        </joint>
+        <link name="${prefix}_ankle_roll_link">
+            <visual>
+                <origin xyz="0.075 0 -0.02"/>
+                <geometry>
+                    <box size="0.3 0.1 0.02" />
+                </geometry>
+                <material name="green" />
+            </visual>
+        </link>
+        <joint name="${prefix}_ankle_roll" type="revolute">
+            <axis xyz="1 0 0" />
+            <limit effort="5.0" lower="-${pi/3}" upper="${pi/3}" velocity="5.0" />
+            <origin xyz="0 0 0" rpy="0 0 0" />
+            <parent link="${prefix}_ankle_pitch_link" />
+            <child link="${prefix}_ankle_roll_link" />
+        </joint>
+    </xacro:macro>
+    <xacro:macro name="biped_left_leg" params="parent_link">
+        <xacro:biped_leg prefix="l" parent_link="${parent_link}" reflect="1" />
+    </xacro:macro>
+    <xacro:macro name="biped_right_leg" params="parent_link">
+        <xacro:biped_leg prefix="r" parent_link="${parent_link}" reflect="-1" />
+    </xacro:macro>
+    <xacro:biped_left_leg parent_link="base_link" />
+    <xacro:biped_right_leg parent_link="base_link" />
 </robot>

Commit message: Fix leg link visual

File: biped_description/urdf/biped.urdf.xacro (robot description, xacro)
@@ -25,5 +25,5 @@
         <link name="${prefix}_pelvis_pitch_link">
             <visual>
-                <origin xyz="0 0 -0.20"/>
+                <origin xyz="0 0 -0.25"/>
                 <geometry>
                     <cylinder radius="0.02" length="0.5" />

Commit message: Change joint limits

File: biped_description/urdf/biped.urdf.xacro (robot description, xacro)
@@ -34,5 +34,5 @@
         <joint name="${prefix}_pelvis_yaw" type="revolute">
             <axis xyz="0 0 1" />
-            <limit effort="5.0" lower="-${pi/3}" upper="${pi/3}" velocity="5.0" />
+            <limit effort="10.0" lower="-${pi/3}" upper="${pi/3}" velocity="50.00" />
             <origin xyz="0 ${reflect*0.25} 0" rpy="0 0 0" />
             <parent link="${parent_link}" />
@@ -41,5 +41,5 @@
         <joint name="${prefix}_pelvis_roll" type="revolute">
             <axis xyz="1 0 0" />
-            <limit effort="5.0" lower="-${pi/3}" upper="${pi/3}" velocity="5.0" />
+            <limit effort="10.0" lower="-${pi/3}" upper="${pi/3}" velocity="50.0" />
             <origin xyz="0 0 0" rpy="0 0 0" />
             <parent link="${prefix}_pelvis_yaw_link" />
@@ -48,5 +48,5 @@
         <joint name="${prefix}_pelvis_pitch" type="revolute">
             <axis xyz="0 1 0" />
-            <limit effort="5.0" lower="-${pi/3}" upper="${pi/3}" velocity="5.0" />
+            <limit effort="10.0" lower="-${pi/3}" upper="${pi/3}" velocity="50.0" />
             <origin xyz="0 0 0" rpy="0 0 0" />
             <parent link="${prefix}_pelvis_roll_link" />
@@ -64,5 +64,5 @@
         <joint name="${prefix}_knee_pitch" type="revolute">
             <axis xyz="0 1 0" />
-            <limit effort="5.0" lower="0" upper="${pi/2}" velocity="5.0" />
+            <limit effort="10.0" lower="0" upper="${pi/2}" velocity="50.0" />
             <origin xyz="0 0 -0.5" rpy="0 0 0" />
             <parent link="${prefix}_pelvis_pitch_link" />
@@ -73,5 +73,5 @@
         <joint name="${prefix}_ankle_pitch" type="revolute">
             <axis xyz="0 1 0" />
-            <limit effort="5.0" lower="-${pi/3}" upper="${pi/3}" velocity="5.0" />
+            <limit effort="10.0" lower="-${pi/3}" upper="${pi/3}" velocity="50.0" />
             <origin xyz="0 0 -0.5" rpy="0 0 0" />
             <parent link="${prefix}_knee_pitch_link" />
@@ -89,5 +89,5 @@
         <joint name="${prefix}_ankle_roll" type="revolute">
             <axis xyz="1 0 0" />
-            <limit effort="5.0" lower="-${pi/3}" upper="${pi/3}" velocity="5.0" />
+            <limit effort="10.0" lower="-${pi/3}" upper="${pi/3}" velocity="50.0" />
             <origin xyz="0 0 0" rpy="0 0 0" />
             <parent link="${prefix}_ankle_pitch_link" />

Commit message: Fix urdf_joint_limits segfault : ^ )
Always check your pointers

File: biped_description/urdf/biped.urdf.xacro (robot description, xacro)
@@ -94,4 +94,11 @@
             <child link="${prefix}_ankle_roll_link" />
         </joint>
+        <link name="${prefix}_ankle">
+        </link>
+        <joint name="${prefix}_ankle_fixed" type="fixed">
+            <origin xyz="0 0 0" rpy="0 0 0" />
+            <parent link="${prefix}_ankle_roll_link" />
+            <child link="${prefix}_ankle" />
+        </joint>
     </xacro:macro>
     <xacro:macro name="biped_left_leg" params="parent_link">

Commit message: Add collision meshes

File: biped_description/urdf/biped.urdf.xacro (robot description, xacro)
@@ -26,9 +26,15 @@
             <visual>
                 <origin xyz="0 0 -0.25"/>
+                <material name="blue"/>
                 <geometry>
                     <cylinder radius="0.02" length="0.5" />
                 </geometry>
-                <material name="blue"/>
             </visual>
+            <collision>
+                <origin xyz="0 0 -0.25"/>
+                <geometry>
+                    <cylinder radius="0.02" length="0.5"/>
+                </geometry>
+            </collision>
         </link>
         <joint name="${prefix}_pelvis_yaw" type="revolute">
@@ -61,4 +67,10 @@
                 <material name="red"/>
             </visual>
+            <collision>
+                <origin xyz="0 0 -0.25"/>
+                <geometry>
+                    <cylinder radius="0.02" length="0.5" />
+                </geometry>
+            </collision>
         </link>
         <joint name="${prefix}_knee_pitch" type="revolute">
@@ -86,4 +98,10 @@
                 <material name="green" />
             </visual>
+            <collision>
+                <origin xyz="0.075 0 -0.02"/>
+                <geometry>
+                    <box size="0.3 0.1 0.02" />
+                </geometry>
+            </collision>
         </link>
         <joint name="${prefix}_ankle_roll" type="revolute">
