Commit message: Add inertial parameters and base_footprint frame

File: biped_description/urdf/biped.urdf.xacro (robot description, xacro)
@@ -1,4 +1,5 @@
 <?xml version="1.0"?>
 <robot xmlns:xacro="http://www.ros.org/wiki/xacro" name="biped">
+    <gazebo />
     <material name="red">
         <color rgba="0.8 0 0 1"/>
@@ -16,10 +17,48 @@
         <color rgba="0 0 0 1" />
     </material>
+    <xacro:macro name="empty_inertial" params="">
+        <inertial>
+            <mass value="0.0" />
+            <inertia
+                    ixx="0.0" ixy="0.0" ixz="0.0"
+                    iyy="0.0" iyz="0.0"
+                    izz="0.0" />
+        </inertial>
+    </xacro:macro>
+    <xacro:macro name="cylinder_inertial" params="r l m">
+        <inertial>
+            <mass value="${m}" />
+            <inertia
+                    ixx="${(1.0/12.0)*m*(3.0*r*r + l*l)}" ixy="0.0" ixz="0.0"
+                    iyy="${(1.0/12.0)*m*(3.0*r*r + l*l)}" iyz="0.0"
+                    izz="${(1.0/2.0)*m*r*r}" />
+        </inertial>
+    </xacro:macro>
+    <xacro:macro name="box_inertial" params="w h d m">
+        <inertial>
+            <mass value="${m}" />
+            <inertia
+                    ixx="${(1.0/12.0)*m*(h*h + d*d)}" ixy="0.0" ixz="0.0"
+                    iyy="${(1.0/12.0)*m*(w*w + d*d)}" iyz="0.0"
+                    izz="${(1.0/12.0)*m*(w*w + h*h)}" />
+        </inertial>
+    </xacro:macro>
+    <link name="base_footprint">
+        <xacro:empty_inertial />
+    </link>
     <link name="base_link">
+        <xacro:empty_inertial />
     </link>
+    <joint name="footprint_to_waist" type="fixed">
+        <origin xyz="0 0 1.0" />
+        <parent link="base_footprint" />
+        <child link="base_link" />
+    </joint>
     <xacro:macro name="biped_leg" params="parent_link prefix reflect">
         <link name="${prefix}_pelvis_yaw_link">
+            <xacro:empty_inertial />
         </link>
         <link name="${prefix}_pelvis_roll_link">
+            <xacro:empty_inertial />
         </link>
         <link name="${prefix}_pelvis_pitch_link">
@@ -37,8 +76,9 @@
                 </geometry>
             </collision>
+            <xacro:cylinder_inertial r="0.02" l="0.5" m="0.25"/>
         </link>
         <joint name="${prefix}_pelvis_yaw" type="revolute">
             <axis xyz="0 0 1" />
-            <limit effort="10.0" lower="-${pi/3}" upper="${pi/3}" velocity="50.00" />
+            <limit effort="10.0" lower="-${pi/3}" upper="${pi/3}" velocity="5.00" />
             <origin xyz="0 ${reflect*0.25} 0" rpy="0 0 0" />
             <parent link="${parent_link}" />
@@ -47,5 +87,5 @@
         <joint name="${prefix}_pelvis_roll" type="revolute">
             <axis xyz="1 0 0" />
-            <limit effort="10.0" lower="-${pi/3}" upper="${pi/3}" velocity="50.0" />
+            <limit effort="10.0" lower="-${pi/3}" upper="${pi/3}" velocity="5.0" />
             <origin xyz="0 0 0" rpy="0 0 0" />
             <parent link="${prefix}_pelvis_yaw_link" />
@@ -54,5 +94,5 @@
         <joint name="${prefix}_pelvis_pitch" type="revolute">
             <axis xyz="0 1 0" />
-            <limit effort="10.0" lower="-${pi/3}" upper="${pi/3}" velocity="50.0" />
+            <limit effort="10.0" lower="-${pi/3}" upper="${pi/3}" velocity="5.0" />
             <origin xyz="0 0 0" rpy="0 0 0" />
             <parent link="${prefix}_pelvis_roll_link" />
@@ -73,8 +113,9 @@
                 </geometry>
             </collision>
+            <xacro:cylinder_inertial r="0.02" l="0.5" m="0.25"/>
         </link>
         <joint name="${prefix}_knee_pitch" type="revolute">
             <axis xyz="0 1 0" />
-            <limit effort="10.0" lower="0" upper="${pi/2}" velocity="50.0" />
+            <limit effort="10.0" lower="0" upper="${pi/2}" velocity="5.0" />
             <origin xyz="0 0 -0.5" rpy="0 0 0" />
             <parent link="${prefix}_pelvis_pitch_link" />
@@ -82,8 +123,9 @@
         </joint>
         <link name="${prefix}_ankle_pitch_link">
+            <xacro:empty_inertial />
         </link>
         <joint name="${prefix}_ankle_pitch" type="revolute">
             <axis xyz="0 1 0" />
-            <limit effort="10.0" lower="-${pi/3}" upper="${pi/3}" velocity="50.0" />
+            <limit effort="10.0" lower="-${pi/3}" upper="${pi/3}" velocity="5.0" />
             <origin xyz="0 0 -0.5" rpy="0 0 0" />
             <parent link="${prefix}_knee_pitch_link" />
@@ -104,8 +146,9 @@
                 </geometry>
             </collision>
+            <xacro:box_inertial w="0.3" h="0.1" d="0.02" m="0.1"/>
         </link>
         <joint name="${prefix}_ankle_roll" type="revolute">
             <axis xyz="1 0 0" />
-            <limit effort="10.0" lower="-${pi/3}" upper="${pi/3}" velocity="50.0" />
+            <limit effort="10.0" lower="-${pi/3}" upper="${pi/3}" velocity="5.0" />
             <origin xyz="0 0 0" rpy="0 0 0" />
             <parent link="${prefix}_ankle_pitch_link" />
@@ -113,4 +156,5 @@
         </joint>
         <link name="${prefix}_ankle">
+            <xacro:empty_inertial />
         </link>
         <joint name="${prefix}_ankle_fixed" type="fixed">

Commit message: Change footprint_to_waist joint name to footprint_fixed

File: biped_description/urdf/biped.urdf.xacro (robot description, xacro)
@@ -50,5 +50,5 @@
         <xacro:empty_inertial />
     </link>
-    <joint name="footprint_to_waist" type="fixed">
+    <joint name="footprint_fixed" type="fixed">
         <origin xyz="0 0 1.0" />
         <parent link="base_footprint" />

Commit message: Trying to fix gazebo bounding box error

File: biped_description/urdf/biped.urdf.xacro (robot description, xacro)
@@ -1,4 +1,4 @@
 <?xml version="1.0"?>
-<robot xmlns:xacro="http://www.ros.org/wiki/xacro" name="biped">
+<robot name="biped" xmlns:xacro="http://www.ros.org/wiki/xacro">
     <material name="red">
         <color rgba="0.8 0 0 1"/>
@@ -20,8 +20,22 @@
             <mass value="0.0" />
             <inertia
-                    ixx="0.0" ixy="0.0" ixz="0.0"
-                    iyy="0.0" iyz="0.0"
-                    izz="0.0" />
+                    ixx="1.0" ixy="0.0" ixz="0.0"
+                    iyy="1.0" iyz="0.0"
+                    izz="1.0" />
         </inertial>
+    </xacro:macro>
+    <xacro:macro name="empty_gazebo_link" params="">
+        <visual>
+            <geometry>
+                <box size="0.001 0.001 0.001"/>
+            </geometry>
+            <material name="black" />
+        </visual>
+        <collision>
+            <geometry>
+                <box size="0.001 0.001 0.001"/>
+            </geometry>
+        </collision>
+        <xacro:empty_inertial />
     </xacro:macro>
     <xacro:macro name="cylinder_inertial" params="r l m">
@@ -43,21 +57,32 @@
         </inertial>
     </xacro:macro>
-    <link name="base_footprint">
-        <xacro:empty_inertial />
+    <link name="base_link">
+        <xacro:empty_gazebo_link />
     </link>
-    <link name="base_link">
-        <xacro:empty_inertial />
+    <link name="waist_link">
+        <xacro:empty_gazebo_link />
     </link>
-    <joint name="footprint_fixed" type="fixed">
+    <joint name="base_fixed" type="fixed">
+        <parent link="base_link" />
+        <child link="waist_link" />
         <origin xyz="0 0 1.0" />
-        <parent link="base_footprint" />
-        <child link="base_link" />
     </joint>
+    <xacro:macro name="revolute_transmission" params="joint_name reduction">
+        <transmission name="${joint_name}_trans">
+            <type>transmission_interface/SimpleTransmission</type>
+            <actuator name="${joint_name}_motor">
+                <mechanicalReduction>${reduction}</mechanicalReduction>
+            </actuator>
+            <joint name="${joint_name}">
+                <hardwareInterface>hardware_interface/PositionJointInterface</hardwareInterface>
+            </joint>
+        </transmission>
+    </xacro:macro>
     <xacro:macro name="biped_leg" params="parent_link prefix reflect">
         <link name="${prefix}_pelvis_yaw_link">
-            <xacro:empty_inertial />
+            <xacro:empty_gazebo_link />
         </link>
         <link name="${prefix}_pelvis_roll_link">
-            <xacro:empty_inertial />
+            <xacro:empty_gazebo_link />
         </link>
         <link name="${prefix}_pelvis_pitch_link">
@@ -78,23 +103,23 @@
         </link>
         <joint name="${prefix}_pelvis_yaw" type="revolute">
-            <axis xyz="0 0 1" />
-            <limit effort="10.0" lower="-${pi/3}" upper="${pi/3}" velocity="5.00" />
-            <origin xyz="0 ${reflect*0.25} 0" rpy="0 0 0" />
             <parent link="${parent_link}" />
             <child link="${prefix}_pelvis_yaw_link" />
+            <axis xyz="0 0 1" />
+            <origin xyz="0 ${reflect*0.25} 0" rpy="0 0 0" />
+            <limit effort="10.0" lower="-${pi/3}" upper="${pi/3}" velocity="5.00" />
         </joint>
         <joint name="${prefix}_pelvis_roll" type="revolute">
-            <axis xyz="1 0 0" />
-            <limit effort="10.0" lower="-${pi/3}" upper="${pi/3}" velocity="5.0" />
-            <origin xyz="0 0 0" rpy="0 0 0" />
             <parent link="${prefix}_pelvis_yaw_link" />
             <child link="${prefix}_pelvis_roll_link" />
+            <axis xyz="1 0 0" />
+            <origin xyz="0 0 0" rpy="0 0 0" />
+            <limit effort="10.0" lower="-${pi/3}" upper="${pi/3}" velocity="5.0" />
         </joint>
         <joint name="${prefix}_pelvis_pitch" type="revolute">
-            <axis xyz="0 1 0" />
-            <limit effort="10.0" lower="-${pi/3}" upper="${pi/3}" velocity="5.0" />
-            <origin xyz="0 0 0" rpy="0 0 0" />
             <parent link="${prefix}_pelvis_roll_link" />
             <child link="${prefix}_pelvis_pitch_link" />
+            <axis xyz="0 1 0" />
+            <origin xyz="0 0 0" rpy="0 0 0" />
+            <limit effort="10.0" lower="-${pi/3}" upper="${pi/3}" velocity="5.0" />
         </joint>
         <link name="${prefix}_knee_pitch_link">
@@ -115,20 +140,13 @@
         </link>
         <joint name="${prefix}_knee_pitch" type="revolute">
-            <axis xyz="0 1 0" />
-            <limit effort="10.0" lower="0" upper="${pi/2}" velocity="5.0" />
-            <origin xyz="0 0 -0.5" rpy="0 0 0" />
             <parent link="${prefix}_pelvis_pitch_link" />
             <child link="${prefix}_knee_pitch_link" />
+            <axis xyz="0 1 0" />
+            <origin xyz="0 0 -0.5" rpy="0 0 0" />
+            <limit effort="10.0" lower="0" upper="${pi/2}" velocity="5.0" />
         </joint>
         <link name="${prefix}_ankle_pitch_link">
-            <xacro:empty_inertial />
-        </link>
-        <joint name="${prefix}_ankle_pitch" type="revolute">
-            <axis xyz="0 1 0" />
-            <limit effort="10.0" lower="-${pi/3}" upper="${pi/3}" velocity="5.0" />
-            <origin xyz="0 0 -0.5" rpy="0 0 0" />
-            <parent link="${prefix}_knee_pitch_link" />
-            <child link="${prefix}_ankle_pitch_link" />
-        </joint>
+            <xacro:empty_gazebo_link />
+        </link>
         <link name="${prefix}_ankle_roll_link">
             <visual>
@@ -147,19 +165,31 @@
             <xacro:box_inertial w="0.3" h="0.1" d="0.02" m="0.1"/>
         </link>
+        <joint name="${prefix}_ankle_pitch" type="revolute">
+            <parent link="${prefix}_knee_pitch_link" />
+            <child link="${prefix}_ankle_pitch_link" />
+            <axis xyz="0 1 0" />
+            <origin xyz="0 0 -0.5" rpy="0 0 0" />
+            <limit effort="10.0" lower="-${pi/3}" upper="${pi/3}" velocity="5.0" />
+        </joint>
         <joint name="${prefix}_ankle_roll" type="revolute">
-            <axis xyz="1 0 0" />
-            <limit effort="10.0" lower="-${pi/3}" upper="${pi/3}" velocity="5.0" />
-            <origin xyz="0 0 0" rpy="0 0 0" />
             <parent link="${prefix}_ankle_pitch_link" />
             <child link="${prefix}_ankle_roll_link" />
+            <axis xyz="1 0 0" />
+            <origin xyz="0 0 0" rpy="0 0 0" />
+            <limit effort="10.0" lower="-${pi/3}" upper="${pi/3}" velocity="5.0" />
         </joint>
         <link name="${prefix}_ankle">
-            <xacro:empty_inertial />
+            <xacro:empty_gazebo_link />
         </link>
         <joint name="${prefix}_ankle_fixed" type="fixed">
-            <origin xyz="0 0 0" rpy="0 0 0" />
             <parent link="${prefix}_ankle_roll_link" />
             <child link="${prefix}_ankle" />
         </joint>
+        <xacro:revolute_transmission joint_name="${prefix}_pelvis_yaw" reduction="1" />
+        <xacro:revolute_transmission joint_name="${prefix}_pelvis_roll" reduction="1" />
+        <xacro:revolute_transmission joint_name="${prefix}_pelvis_pitch" reduction="1" />
+        <xacro:revolute_transmission joint_name="${prefix}_knee_pitch" reduction="1" />
+        <xacro:revolute_transmission joint_name="${prefix}_ankle_pitch" reduction="1" />
+        <xacro:revolute_transmission joint_name="${prefix}_ankle_roll" reduction="1" />
     </xacro:macro>
     <xacro:macro name="biped_left_leg" params="parent_link">
@@ -169,6 +199,6 @@
         <xacro:biped_leg prefix="r" parent_link="${parent_link}" reflect="-1" />
     </xacro:macro>
-    <xacro:biped_left_leg parent_link="base_link" />
-    <xacro:biped_right_leg parent_link="base_link" />
+    <xacro:biped_left_leg parent_link="waist_link" />
+    <xacro:biped_right_leg parent_link="waist_link" />
     <gazebo>
         <plugin name="gazebo_ros_control" filename="libgazebo_ros_control.so">

Commit message: Working gazebo simulation
Don't set mass=0.0 :^)

File: biped_description/urdf/biped.urdf.xacro (robot description, xacro)
@@ -18,9 +18,9 @@
     <xacro:macro name="empty_inertial" params="">
         <inertial>
-            <mass value="0.0" />
+            <mass value="0.0001" />
             <inertia
-                    ixx="1.0" ixy="0.0" ixz="0.0"
-                    iyy="1.0" iyz="0.0"
-                    izz="1.0" />
+                    ixx="0.0001" ixy="0.0" ixz="0.0"
+                    iyy="0.0001" iyz="0.0"
+                    izz="0.0001" />
         </inertial>
     </xacro:macro>
@@ -28,13 +28,8 @@
         <visual>
             <geometry>
-                <box size="0.001 0.001 0.001"/>
+                <sphere radius="0.01"/>
             </geometry>
-            <material name="black" />
+            <material name="red" />
         </visual>
-        <collision>
-            <geometry>
-                <box size="0.001 0.001 0.001"/>
-            </geometry>
-        </collision>
         <xacro:empty_inertial />
     </xacro:macro>
@@ -75,5 +70,5 @@
             </actuator>
             <joint name="${joint_name}">
-                <hardwareInterface>hardware_interface/PositionJointInterface</hardwareInterface>
+                <hardwareInterface>hardware_interface/EffortJointInterface</hardwareInterface>
             </joint>
         </transmission>
@@ -107,5 +102,5 @@
             <axis xyz="0 0 1" />
             <origin xyz="0 ${reflect*0.25} 0" rpy="0 0 0" />
-            <limit effort="10.0" lower="-${pi/3}" upper="${pi/3}" velocity="5.00" />
+            <limit effort="10.0" lower="-${pi/3}" upper="${pi/3}" velocity="5.0" />
         </joint>
         <joint name="${prefix}_pelvis_roll" type="revolute">
@@ -203,5 +198,5 @@
     <gazebo>
         <plugin name="gazebo_ros_control" filename="libgazebo_ros_control.so">
-            <robotNamespace>/</robotNamespace>
+            <robotNamespace>/biped</robotNamespace>
         </plugin>
     </gazebo>

Commit message: Add foot friction and IMU

File: biped_description/urdf/biped.urdf.xacro (robot description, xacro)
@@ -52,13 +52,33 @@
         </inertial>
     </xacro:macro>
-    <link name="base_link">
+    <link name="base_link" />
+    <link name="torso_link">
+         <visual>
+            <origin xyz="0 0 0" rpy="0 0 0" />
+            <geometry>
+                <box size="0.1 0.7 0.7"/>
+            </geometry>
+            <material name="red" />
+        </visual>
+        <collision>
+            <origin xyz="0 0 0" rpy="0 0 0" />
+            <geometry>
+                <box size="0.1 0.7 0.7"/>
+            </geometry>
+        </collision>
+        <xacro:box_inertial w="0.1" h="0.7" d="0.7" m="2.0" />
     </link>
-    <link name="waist_link">
+    <joint name="torso_fixed" type="fixed">
+        <origin xyz="0 0 0.35" rpy="0 0 0" />
+        <parent link="base_link"/>
+        <child link="torso_link" />
+    </joint>
+    <link name="imu_link">
         <xacro:empty_gazebo_link />
     </link>
-    <joint name="base_fixed" type="fixed">
-        <parent link="base_link" />
-        <child link="waist_link" />
-        <origin xyz="0 0 1.0" />
+    <joint name="imu_fixed" type="fixed">
+        <origin xyz="0 0 0" rpy="0 0 0" />
+        <parent link="torso_link" />
+        <child link="imu_link" />
     </joint>
     <xacro:macro name="revolute_transmission" params="joint_name reduction">
@@ -193,6 +213,6 @@
         <xacro:biped_leg prefix="r" parent_link="${parent_link}" reflect="-1" />
     </xacro:macro>
-    <xacro:biped_left_leg parent_link="waist_link" />
-    <xacro:biped_right_leg parent_link="waist_link" />
+    <xacro:biped_left_leg parent_link="base_link" />
+    <xacro:biped_right_leg parent_link="base_link" />
     <gazebo>
         <plugin name="gazebo_ros_control" filename="libgazebo_ros_control.so">
@@ -201,3 +221,43 @@
         </plugin>
     </gazebo>
+    <gazebo reference="l_ankle_roll_link">
+        <material>Gazebo/FlatBlack</material>
+        <kp>1000000.0</kp>
+        <kd>100.0</kd>
+        <mu1>1.0</mu1>
+        <mu2>1.0</mu2>
+        <fdir1>1 0 0</fdir1>
+        <maxVel>1.0</maxVel>
+        <minDepth>0.0</minDepth>
+    </gazebo>
+    <gazebo reference="r_ankle_roll_link">
+        <material>Gazebo/FlatBlack</material>
+        <kp>1000000.0</kp>
+        <kd>100.0</kd>
+        <mu1>1.0</mu1>
+        <mu2>1.0</mu2>
+        <fdir1>1 0 0</fdir1>
+        <maxVel>1.0</maxVel>
+        <minDepth>0.0</minDepth>
+    </gazebo>
+    <gazebo reference="imu_link">
+        <gravity>true</gravity>
+        <sensor name="imu_sensor" type="imu">
+            <always_on>true</always_on>
+            <update_rate>100</update_rate>
+            <visualize>true</visualize>
+            <topic>__default_topic__</topic>
+            <plugin filename="libgazebo_ros_imu_sensor.so" name="imu_plugin">
+                <robotNamespace>/biped</robotNamespace>
+                <topicName>imu</topicName>
+                <bodyName>imu_link</bodyName>
+                <updateRateHZ>10</updateRateHZ>
+                <gaussianNoise>0.0</gaussianNoise>
+                <xyzOffset>0 0 0</xyzOffset>
+                <rpyOffset>0 0 0</rpyOffset>
+                <frameName>imu_link</frameName>
+            </plugin>
+            <pose>0 0 0 0 0 0</pose>
+        </sensor>
+    </gazebo>
 </robot>
